File: tests/board_samples/kicad_8/kicad_bom_1.kicad_sch (KiCad schematic)
At the start: 6 parts

Commit message: [BoM][Adde] "KICAD" format
- This is some sort of configurable CSV
- We get the options from the project
Parts:
- R2: now in the parts list
Changed lines of the file:
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@@
 		(on_board yes)
 		(dnp no)
-		(fields_autoplaced yes)
 		(property "Reference" "R1"
 			(at 38.1 63.4999 0)
@@
 			)
 		)
-		(property "Description" "Resistor"
-			(at 35.56 64.77 0)
-			(effects
-				(font
-					(size 1.27 1.27)
-				)
-				(hide yes)
+		(property "Description" "Resistor\"\n	Hola"
+			(at 35.814 70.612 0)
+			(effects
+				(font
+					(size 1.27 1.27)
+				)
 			)
 		)
@@
 		(unit 1)
 		(exclude_from_sim no)
-		(in_bom no)
-		(on_board yes)
-		(dnp no)
+		(in_bom yes)
+		(on_board yes)
+		(dnp no)
