File: tests/board_samples/kicad_9/light_control_diff.kicad_pcb (KiCad board)
At the start: 4 copper layers, 59.7 x 48.3 mm, 77 parts, among them J1 Screw_Terminal_01x02, J10 Screw_Terminal_01x02, J11 Screw_Terminal_01x02, J12 Conn_01x03, J2 USB_B_Micro, J3 Screw_Terminal_01x02, J4 Screw_Terminal_01x02, J5 Screw_Terminal_01x02, J6 Screw_Terminal_01x02, J7 Screw_Terminal_01x02, J8 Screw_Terminal_01x02, J9 Screw_Terminal_01x02, Q1 Q_NPN_BEC, Q10 Q_NMOS_GDS, Q2 Q_NPN_BEC, Q3 Q_NMOS_GSD, Q4 Q_NMOS_GDS, Q5 Q_NMOS_GDS, Q6 Q_NMOS_GDS, Q7 Q_NMOS_GDS, Q8 Q_NMOS_GDS, Q9 Q_NMOS_GDS, SW1 SW_Push, U1 AZ1117-3.3, U2 CP2104, U3 ESP32-WROOM-32, U4 DHT11

Commit message: [Tests][Added][KiCad 9] SCH and PCB examples
Parts:
- C6: value 4.7uF -> 0.1uF
Other:
- board text added: "WiredHut Light Control / Temperature Humidity Sensor"
- board text removed: "WiredHut ${gh} ${date} Light Control / Temperature Humidity Sensor"
